Commit message: Add files via upload

File: ros2_control_demo_description/goliath/urdf/goliath_description.urdf.xacro (robot description, xacro)
@@ -8,4 +8,5 @@
       xyz_offset="0 0 0"
       rpy_offset="0 0 0"
+      material="silver"
       mesh_package="ros2_control_demo_description/goliath"
       mesh_name="link_0"
@@ -15,4 +16,5 @@
       xyz_offset="0 0 0"
       rpy_offset="0 0 0"
+      material="silver"
       mesh_package="ros2_control_demo_description/goliath"
       mesh_name="link_1"
@@ -22,4 +24,5 @@
       xyz_offset="0 0 0"
       rpy_offset="0 0 0"
+      material="silver"
       mesh_package="ros2_control_demo_description/goliath"
       mesh_name="link_2"
@@ -29,4 +32,5 @@
       xyz_offset="0 0 0"
       rpy_offset="0 0 0"
+      material="silver"
       mesh_package="ros2_control_demo_description/goliath"
       mesh_name="link_3"
@@ -36,4 +40,5 @@
       xyz_offset="0 0 0"
       rpy_offset="0 0 0"
+      material="silver"
       mesh_package="ros2_control_demo_description/goliath"
       mesh_name="link_4"
@@ -43,4 +48,5 @@
       xyz_offset="0 0 0"
       rpy_offset="0 0 0"
+      material="silver"
       mesh_package="ros2_control_demo_description/goliath"
       mesh_name="link_5"
@@ -48,12 +54,152 @@
   <xacro:create_link
       link_name="link_6"
-      xyz_offset="0 0 0"
-      rpy_offset="0 0 0"
-      mesh_package="ros2_control_demo_description/goliath"
-      mesh_name="link_6"
-  />
-  <link name="ft_frame"/>
-  <link name="tool0"/>
-  <!-- base_joint fixes base_link to the environment -->
+      xyz_offset="0.006 -0.009 0.006"
+      rpy_offset="0 0 1.5775"
+      material="silver"
+      mesh_package="ros2_control_demo_description/goliath"
+      mesh_name="tool_connector"
+  />
+<xacro:create_link
+      link_name="tool_connector"
+      xyz_offset="-0.0036 0.0053 0.0176"
+      rpy_offset="0 0 0"
+      material="silver"
+      mesh_package="ros2_control_demo_description/goliath"
+      mesh_name="tool_base"
+  />
+ <!--  ++++++++++++++++++++++++++++++++++++++++++++++++++++++++++++++++++++++++++++++++
+            tool_links - change out the tool here (optional)
+       ++++++++++++++++++++++++++++++++++++++++++++++++++++++++++++++++++++++++++++++++     -->
+<xacro:create_link
+      link_name="tool_base"
+      xyz_offset="0 0 0"
+      rpy_offset="0 0 0"
+      material="silver"
+      mesh_package="ros2_control_demo_description/goliath"
+      mesh_name="tool_base"
+  />
+  <link name="grip_mount_1">
+  <inertial>
+    <origin xyz="-0.00034136005542522146 0.015547767390796129 0.01883273293370806" rpy="0 0 0"/>
+    <mass value="0.026038448039166225"/>
+    <inertia ixx="5e-06" iyy="4e-06" izz="5e-06" ixy="0.0" iyz="-1e-06" ixz="0.0"/>
+  </inertial>
+  <visual>
+    <origin xyz="-0.000365 0.006365 -0.008562" rpy="0 0 0"/>
+    <geometry>
+      <mesh filename="file://$(find gripper_description)/meshes/grip_mount_1.stl" scale="0.001 0.001 0.001"/>
+    </geometry>
+    <material name="black"/>
+  </visual>
+  <collision>
+    <origin xyz="-0.000365 0.006365 -0.008562" rpy="0 0 0"/>
+    <geometry>
+      <mesh filename="file://$(find gripper_description)/meshes/grip_mount_1.stl" scale="0.001 0.001 0.001"/>
+    </geometry>
+  </collision>
+</link>
+<link name="left_mount_1">
+  <inertial>
+    <origin xyz="-0.012312197013134553 0.010499353929422754 0.01616872816060999" rpy="0 0 0"/>
+    <mass value="0.005850260501194334"/>
+    <inertia ixx="1e-06" iyy="1e-06" izz="1e-06" ixy="-0.0" iyz="0.0" ixz="0.0"/>
+  </inertial>
+  <visual>
+    <origin xyz="0.022798 0.016079 -0.032689" rpy="0 0 0"/>
+    <geometry>
+      <mesh filename="file://$(find gripper_description)/meshes/left_mount_1.stl" scale="0.001 0.001 0.001"/>
+    </geometry>
+    <material name="black"/>
+  </visual>
+  <collision>
+    <origin xyz="0.022798 0.016079 -0.032689" rpy="0 0 0"/>
+    <geometry>
+      <mesh filename="file://$(find gripper_description)/meshes/left_mount_1.stl" scale="0.001 0.001 0.001"/>
+    </geometry>
+  </collision>
+</link>
+<link name="right_mount_1">
+  <inertial>
+    <origin xyz="0.012015776314503238 0.010500460176130546 0.016402425646791258" rpy="0 0 0"/>
+    <mass value="0.005851464483284041"/>
+    <inertia ixx="1e-06" iyy="1e-06" izz="1e-06" ixy="0.0" iyz="0.0" ixz="-0.0"/>
+  </inertial>
+  <visual>
+    <origin xyz="-0.022726 0.016079 -0.032981" rpy="0 0 0"/>
+    <geometry>
+      <mesh filename="file://$(find gripper_description)/meshes/right_mount_1.stl" scale="0.001 0.001 0.001"/>
+    </geometry>
+    <material name="black"/>
+  </visual>
+  <collision>
+    <origin xyz="-0.022726 0.016079 -0.032981" rpy="0 0 0"/>
+    <geometry>
+      <mesh filename="file://$(find gripper_description)/meshes/right_mount_1.stl" scale="0.001 0.001 0.001"/>
+    </geometry>
+  </collision>
+</link>
+<link name="rubber_left_1">
+  <inertial>
+    <origin xyz="0.004252295929468346 4.91084999865686e-07 0.02544337370871609" rpy="0 0 0"/>
+    <mass value="0.008265327612092782"/>
+    <inertia ixx="3e-06" iyy="3e-06" izz="1e-06" ixy="-0.0" iyz="-0.0" ixz="-0.0"/>
+  </inertial>
+  <visual>
+    <origin xyz="0.037938 0.005589 -0.06038" rpy="0 0 0"/>
+    <geometry>
+      <mesh filename="file://$(find gripper_description)/meshes/rubber_left_1.stl" scale="0.001 0.001 0.001"/>
+    </geometry>
+    <material name="blue"/>
+  </visual>
+  <collision>
+    <origin xyz="0.037938 0.005589 -0.06038" rpy="0 0 0"/>
+    <geometry>
+      <mesh filename="file://$(find gripper_description)/meshes/rubber_left_1.stl" scale="0.001 0.001 0.001"/>
+    </geometry>
+  </collision>
+</link>
+<link name="rubber_right_1">
+  <inertial>
+    <origin xyz="-0.005023147767699666 4.5740402191025986e-07 0.025301746998458823" rpy="0 0 0"/>
+    <mass value="0.008265327612092756"/>
+    <inertia ixx="3e-06" iyy="3e-06" izz="1e-06" ixy="-0.0" iyz="0.0" ixz="1e-06"/>
+  </inertial>
+  <visual>
+    <origin xyz="-0.036906 0.005579 -0.061218" rpy="0 0 0"/>
+    <geometry>
+      <mesh filename="file://$(find gripper_description)/meshes/rubber_right_1.stl" scale="0.001 0.001 0.001"/>
+    </geometry>
+    <material name="blue"/>
+  </visual>
+  <collision>
+    <origin xyz="-0.036906 0.005579 -0.061218" rpy="0 0 0"/>
+    <geometry>
+      <mesh filename="file://$(find gripper_description)/meshes/rubber_right_1.stl" scale="0.001 0.001 0.001"/>
+    </geometry>
+  </collision>
+</link>
+<link name="t_shirt_1">
+  <inertial>
+    <origin xyz="0.00012163162070136035 -0.009411539665347687 0.013485226893769523" rpy="0 0 0"/>
+    <mass value="0.0026146856075812087"/>
+    <inertia ixx="0.0" iyy="1e-06" izz="0.0" ixy="0.0" iyz="0.0" ixz="-0.0"/>
+  </inertial>
+  <visual>
+    <origin xyz="0.000191 0.007667 -0.022124" rpy="0 0 0"/>
+    <geometry>
+      <mesh filename="file://$(find gripper_description)/meshes/t_shirt_1.stl" scale="0.001 0.001 0.001"/>
+    </geometry>
+    <material name="black"/>
+  </visual>
+  <collision>
+    <origin xyz="0.000191 0.007667 -0.022124" rpy="0 0 0"/>
+    <geometry>
+      <mesh filename="file://$(find gripper_description)/meshes/t_shirt_1.stl" scale="0.001 0.001 0.001"/>
+    </geometry>
+  </collision>
+</link>
+  <!-- +++++++++++++++++++++++++++++++++++++++++++++++++++++++++++++++++++++++++++++++
+            base_joint fixes base_link to the environment
+       +++++++++++++++++++++++++++++++++++++++++++++++++++++++++++++++++++++++++++++++ -->
   <joint name="base_joint" type="fixed">
     <parent link="world"/>
@@ -101,18 +247,55 @@
     <parent link="link_5"/>
     <child link="link_6"/>
-    <origin xyz="0.07318 0 0.02435" rpy="0 ${pi/2} 0"/>
+    <origin xyz="0.07318 0 0.02" rpy="0 ${pi/2} 0"/>
     <axis xyz="0 0 1"/>
     <limit effort="1000.0" lower="${-pi}" upper="${pi}" velocity="2.5"/>
   </joint>
-  <joint name="joint-ft_frame" type="fixed">
+  <joint name="joint_tool_connector_frame" type="fixed">
     <parent link="link_6"/>
-    <child link="ft_frame"/>
+    <child link="tool_connector"/>
     <origin xyz="0 0 0" rpy="0 0 0"/>
   </joint>
-  <joint name="joint-tool" type="fixed">
-    <parent link="ft_frame"/>
-    <child link="tool0"/>
-    <origin xyz="0 0 0.02" rpy="0 0 0"/>
-  </joint>
+  <!-- +++++++++++++++++++++++++++++++++++++++++++++++++++++++++++++++++++++++++++++++++++++++++
+       joints for the tool - softgripper
+       +++++++++++++++++++++++++++++++++++++++++++++++++++++++++++++++++++++++++++++++++++++++++ -->
+  <joint name="joint_connector_frame" type="fixed">
+    <parent link="tool_connector"/>
+    <child link="tool_base"/>
+    <origin xyz="-0.0038 0.005 0.017" rpy="0 0 0"/>
+  </joint>
+<joint name="Rigid 20" type="fixed">
+  <origin xyz="0.000365 -0.006365 0.008562" rpy="0 0 0"/>
+  <parent link="tool_base"/>
+  <child link="grip_mount_1"/>
+</joint>
+<joint name="Slider 22" type="prismatic">
+  <origin xyz="-0.022607 -0.008412 0.010565" rpy="0 0 0"/>
+  <parent link="t_shirt_1"/>
+  <child link="left_mount_1"/>
+  <axis xyz="0.817033 -0.0 0.576591"/>
+  <limit upper="0.022" lower="-0.003" effort="100" velocity="100"/>
+</joint>
+<joint name="Slider 23" type="prismatic">
+  <origin xyz="0.022917 -0.008412 0.010857" rpy="0 0 0"/>
+  <parent link="t_shirt_1"/>
+  <child link="right_mount_1"/>
+  <axis xyz="0.820609 0.0 -0.57149"/>
+  <limit upper="0.003" lower="-0.022" effort="100" velocity="100"/>
+</joint>
+<joint name="Rigid 24" type="fixed">
+  <origin xyz="-0.01514 0.01049 0.027691" rpy="0 0 0"/>
+  <parent link="left_mount_1"/>
+  <child link="rubber_left_1"/>
+</joint>
+<joint name="Rigid 25" type="fixed">
+  <origin xyz="0.01418 0.0105 0.028237" rpy="0 0 0"/>
+  <parent link="right_mount_1"/>
+  <child link="rubber_right_1"/>
+</joint>
+<joint name="Rigid 26" type="fixed">
+  <origin xyz="-0.000556 -0.001302 0.013562" rpy="0 0 0"/>
+  <parent link="grip_mount_1"/>
+  <child link="t_shirt_1"/>
+</joint>
 </xacro:macro>
 </robot>

Commit message: Update goliath_description.urdf.xacro
Added power_box to URDF

File: ros2_control_demo_description/goliath/urdf/goliath_description.urdf.xacro (robot description, xacro)
@@ -67,4 +67,12 @@
       mesh_package="ros2_control_demo_description/goliath"
       mesh_name="tool_base"
+  />
+ <xacro:create_link
+      link_name="power_box"
+      xyz_offset="0 0 0"
+      rpy_offset="0 0 0"
+      material="silver"
+      mesh_package="ros2_control_demo_description/goliath"
+      mesh_name="power_box"
   />
  <!--  ++++++++++++++++++++++++++++++++++++++++++++++++++++++++++++++++++++++++++++++++
@@ -298,4 +306,13 @@
   <child link="t_shirt_1"/>
 </joint>
+<!-- +++++++++++++++++++++++++++++++++++++++++++++++++++++++++++++++++++++++++++++++++++++++++
+       joints for additional parts - powerbox, camera mount, sansors and so on. add STL to Meshes
+                                follow the create link xacro format
+       +++++++++++++++++++++++++++++++++++++++++++++++++++++++++++++++++++++++++++++++++++++++++ -->
+  <joint name="joint_powebox" type="fixed">
+    <parent link="link_2"/>
+    <child link="power_box"/>
+    <origin xyz="-0.276 0 -0.057" rpy="0 1.5775 0"/>
+  </joint>
 </xacro:macro>
 </robot>
